Commit message: Added updates for gazebo to find the models here

File: astrobee_iss/urdf/model.urdf (robot description, URDF)
Before this commit: robot iss, 1 links, 0 joints
Links:
- link body: geometry collision mesh filename=package://astrobee_iss/meshes/cupola.dae; collision mesh filename=package://astrobee_iss/meshes/eu_lab.dae
